File: hw/board-nRF52840/board-nRF52840.kicad_sch (KiCad schematic)
At the start: 8 parts, among them J1 JST-PH 2.0 / BATTERY, U1 XIAO nRF52840, U2 BMA400

Commit message: Add factory reset button
Parts:
- added SW1: B3U-1000P, Board:SW_SPST_B3U-1000P, symbol Board:SW_Push
Connections:
- net GND: now also SW1.2
- net FACTORY_RESET: now reaches U1.1 (D0)
- net FACTORY_RESET: now also SW1.1
- no-connect marks 12 -> 11
Other:
- note added: "Factory reset / pairing"
- note added: "Hold 5 seconds to erase Matter/Thread user state and reboot."
- note added: "Provisioned Matter setup credentials survive factory reset."
- note added: "SW1: active-low D0 (P0.02); firmware internal pull-up."
- note added: "Unpressed contact is open; no external pull-up or RC load."
Changed lines of the file:
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@@
-(kicad_sch (version 20250114) (generator "eeschema") (generator_version "9.0") (paper "A4") (title_block (title "XIAO nRF52840 / BMA400 SMD Carrier") (date "2026-10-07") (rev "A") (company "nrf-matter-thread-ble-esd") (comment 1 "2-layer direct SMD carrier; protected 1S battery; module-specific underside BAT lands"))
+(kicad_sch (version 20250114) (generator "eeschema") (generator_version "9.0") (paper "A4") (title_block (title "XIAO nRF52840 / BMA400 SMD Carrier") (date "2026-10-18") (rev "B") (company "nrf-matter-thread-ble-esd") (comment 1 "2-layer direct SMD carrier; protected 1S battery; module-specific underside BAT lands"))
 (text "Thread / BLE motion sensor" (at 17.78 15.24 0) (effects (font (size 2.54 2.54) (bold yes)) (justify left)))
 (text "XIAO nRF52840 + BMA400  |  direct SMD mounting" (at 17.78 21.59 0) (effects (font (size 1.27 1.27)) (justify left)))
@@
 (wire (pts (xy 83.82 87.63) (xy 91.44 87.63)) (stroke (width 0) (type default)))
 (label "GND" (at 91.44 87.63 0) (effects (font (size 1.016 1.016)) (justify left bottom)))
-(no_connect (at 38.1 46.99))
 (no_connect (at 38.1 52.07))
 (no_connect (at 38.1 62.23))
@@
 (text "PCB-only: H3-H6 underside SWD access; TP1=3V3 Vref, TP2=GND." (at 17.78 191.77 0) (effects (font (size 1.016 1.016)) (justify left)))
 (sheet_instances (path "/" (page "1"))) (embedded_fonts no)
+(wire (pts (xy 38.1 46.99) (xy 20.32 46.99)) (stroke (width 0) (type default)))
+(label "FACTORY_RESET" (at 20.32 46.99 0) (effects (font (size 1.016 1.016)) (justify left bottom)))
+(text "Factory reset / pairing" (at 147.32 116.84 0) (effects (font (size 1.524 1.524) (bold yes)) (justify left)))
+(symbol (lib_id "Board:SW_Push") (at 167.64 134.62 0) (unit 1) (exclude_from_sim no) (in_bom yes) (on_board yes) (dnp no)(property "Reference" "SW1" (at 167.64 127 0) (effects (font (size 1.27 1.27))))(property "Value" "B3U-1000P" (at 167.64 129.54 0) (effects (font (size 1.27 1.27))))(property "Footprint" "Board:SW_SPST_B3U-1000P" (at 167.64 134.62 0) (effects (font (size 1.27 1.27)) (hide yes)))(property "Datasheet" "https://omronfs.omron.com/en_US/ecb/products/pdf/en-b3u.pdf" (at 167.64 134.62 0) (effects (font (size 1.27 1.27)) (hide yes)))(property "Manufacturer" "OMRON (now Aratas)" (at 167.64 134.62 0) (effects (font (size 1.27 1.27)) (hide yes)))(property "MPN" "B3U-1000P" (at 167.64 134.62 0) (effects (font (size 1.27 1.27)) (hide yes)))(property "Datasheet file" "${KIPRJMOD}/datasheets/omron-b3u.pdf" (at 167.64 134.62 0) (effects (font (size 1.27 1.27)) (hide yes)))(property "Supplier" "DigiKey" (at 167.64 134.62 0) (effects (font (size 1.27 1.27)) (hide yes)))(property "Supplier part number" "SW1020CT-ND" (at 167.64 134.62 0) (effects (font (size 1.27 1.27)) (hide yes)))(property "Purchase URL" "https://www.digikey.com/en/products/detail/aratas-formerly-omron-components/B3U-1000P/1534338" (at 167.64 134.62 0) (effects (font (size 1.27 1.27)) (hide yes)))(pin "1")(pin "2")(instances (project "board-nRF52840" (path "/c5032c3c-d00f-5aaf-a428-6cb786e83767" (reference "SW1") (unit 1)))))
+(wire (pts (xy 162.56 134.62) (xy 142.24 134.62)) (stroke (width 0) (type default)))
+(label "FACTORY_RESET" (at 142.24 134.62 0) (effects (font (size 1.016 1.016)) (justify left bottom)))
+(wire (pts (xy 172.72 134.62) (xy 190.5 134.62)) (stroke (width 0) (type default)))
+(label "GND" (at 190.5 134.62 0) (effects (font (size 1.016 1.016)) (justify left bottom)))
+(text "SW1: active-low D0 (P0.02); firmware internal pull-up." (at 142.24 146.05 0) (effects (font (size 1.016 1.016)) (justify left)))
+(text "Hold 5 seconds to erase Matter/Thread user state and reboot." (at 142.24 151.13 0) (effects (font (size 1.016 1.016)) (justify left)))
+(text "Provisioned Matter setup credentials survive factory reset." (at 142.24 156.21 0) (effects (font (size 1.016 1.016)) (justify left)))
+(text "Unpressed contact is open; no external pull-up or RC load." (at 142.24 161.29 0) (effects (font (size 1.016 1.016)) (justify left)))
 )
