File: hw/board-nRF54L15/board-nRF54L15.kicad_pcb (KiCad board)
At the start: 2 copper layers, 30 x 42 mm, 16 parts, among them J1 JST-PH 2.0 / BATTERY, U1 XIAO nRF54L15, U2 BMA400

Commit message: Add factory reset button
Parts:
- added SW1: B3U-1000P, Board:SW_SPST_B3U-1000P, F.Cu at (51.6, 53.2)
Connections:
- U1 pad 1: unconnected-(U1-D0-Pad1) -> /FACTORY_RESET
Routing:
- net /FACTORY_RESET: track 0.00 -> 2.75 mm
- net /GND: track 14.2 -> 16.6 mm, vias 8 -> 9
Other:
- board text added: "BMA400 / Rev B"
- board text removed: "BMA400 / Rev A"

Commit message: Update PCB
Routing:
- net /VBAT: track 43.8 -> 39.6 mm
- net /ACC_INT1: track 30.8 -> 29.7 mm
Changed lines of the file:
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@@
 			(outputformat 1)
 			(mirror no)
-			(drillshape 1)
+			(drillshape 0)
 			(scaleselection 1)
-			(outputdirectory "")
+			(outputdirectory "mfr/")
 		)
 	)
@@
 	)
 	(segment
-		(start 50.773 77.778646)
-		(end 50.773 62.132)
+		(start 56.523 79.427)
+		(end 56.75 79.2)
 		(width 0.25)
 		(layer "F.Cu")
@@
 	)
 	(segment
-		(start 52.421354 79.427)
-		(end 50.773 77.778646)
+		(start 54.945 57.96)
+		(end 50.773 62.132)
 		(width 0.25)
 		(layer "F.Cu")
@@
 	)
 	(segment
-		(start 53 59.905)
-		(end 53 57.96)
+		(start 56.75 79.2)
+		(end 56.75 78.775)
 		(width 0.25)
 		(layer "F.Cu")
@@
 	)
 	(segment
-		(start 56.75 78.775)
-		(end 56.75 79.2)
+		(start 50.773 62.132)
+		(end 50.773 77.778646)
 		(width 0.25)
 		(layer "F.Cu")
@@
 	)
 	(segment
-		(start 56.75 79.2)
+		(start 52.421354 79.427)
 		(end 56.523 79.427)
 		(width 0.25)
@@
 	)
 	(segment
-		(start 50.773 62.132)
-		(end 53 59.905)
-		(width 0.25)
-		(layer "F.Cu")
-		(net "/ACC_INT1")
-	)
-	(segment
-		(start 53 57.96)
-		(end 55.9175 57.96)
+		(start 55.9175 57.96)
+		(end 54.945 57.96)
 		(width 0.25)
 		(layer "F.Cu")
@@
 	)
 	(segment
-		(start 56.523 79.427)
+		(start 50.773 77.778646)
 		(end 52.421354 79.427)
 		(width 0.25)
@@
 	)
 	(segment
-		(start 63.039 65.4277)
-		(end 63.039 67.25)
-		(width 0.4)
-		(layer "F.Cu")
-		(net "/VBAT")
-	)
-	(segment
-		(start 65 83.1)
-		(end 65 85)
+		(start 69.5 78.6)
+		(end 65 83.1)
 		(width 0.6)
 		(layer "F.Cu")
@@
 	)
 	(segment
-		(start 71.9 78.95)
-		(end 71.9 80.9)
-		(width 0.6)
+		(start 63.039 65.4277)
+		(end 63.039 67.25)
+		(width 0.4)
 		(layer "F.Cu")
 		(net "/VBAT")
 	)
 	(segment
-		(start 71.9 80.9)
-		(end 65 83.1)
+		(start 65 83.1)
+		(end 65 85)
 		(width 0.6)
 		(layer "F.Cu")
@@
 	(segment
 		(start 69.5 76.55)
-		(end 71.9 78.95)
+		(end 69.5 78.6)
 		(width 0.6)
 		(layer "F.Cu")

Commit message: Update PCB
Parts:
- added H7: MountingHole_2.2mm_M2, Board:MountingHole_2.2mm_M2, F.Cu at (52.0, 53.0)
- added H8: MountingHole_2.2mm_M2, Board:MountingHole_2.2mm_M2, F.Cu at (68.0, 53.0)
- C1, C2, C3, R1, R2, U2: moved to B.Cu
- moved H3 22.0 mm to (50.8, 70.2), turned to 90 degrees
- moved H4 21.5 mm to (50.8, 67.7), turned to 90 degrees
- moved H5 18.5 mm to (53.3, 70.2), turned to 90 degrees
- moved H6 17.9 mm to (53.3, 67.7), turned to 90 degrees
- moved C1 11.2 mm to (56.5, 68.8), turned to 180 degrees
- moved U1 9.62 mm to (59.5, 69.0), turned to 90 degrees
- moved U2 9.49 mm to (60.0, 69.0)
- moved H2 8.94 mm to (68.0, 85.0)
- moved SW1 8.71 mm to (60.0, 55.5), turned to 0 degrees
- moved C2 8.38 mm to (63.5, 71.5), turned to 0 degrees
- moved TP1 7.17 mm to (67.5, 81.0)
- moved TP2 7.07 mm to (67.5, 79.0)
- moved C3 6.00 mm to (65.0, 74.0), turned to 180 degrees
- moved R2 6.00 mm to (57.5, 74.0), turned to 0 degrees
- moved J1 5.66 mm to (59.0, 81.0)
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Routing:
- net /FACTORY_RESET: track 2.75 -> 29.8 mm
- net /VBAT: track 39.6 -> 15.5 mm, vias 2 -> 0
- net /+3V3: track 76.6 -> 62.8 mm, vias 6 -> 1
- net /ACC_INT1: track 29.7 -> 21.3 mm, vias 0 -> 1
- net /GND: track 16.6 -> 8.29 mm, vias 9 -> 7
- net /I2C_SCL: track 19.9 -> 17.1 mm, vias 2 -> 1
- net /I2C_SDA: track 19.7 -> 17.7 mm, vias 2 -> 1
Other:
- board size 30 x 42 mm -> 22 x 38 mm
- board text added: "22 x 38 mm / 2 layers / 1.6 mm FR4"
- board text added: "BMA400 / Rev C"
- board text removed: "30 x 42 mm / 2 layers / 1.6 mm FR4"
- board text removed: "BMA400 / Rev B"
